File: kicad/exp60.kicad_pcb (KiCad board)
At the start: 2 copper layers, 285.8 x 95.2 mm, 152 parts, among them J0 USB4105-GF-A, K0 KEYSW, K1 KEYSW, K10 KEYSW, K11 KEYSW, K12 KEYSW, K13 KEYSW, K14 KEYSW, K15 KEYSW, K16 KEYSW, K17 KEYSW, K18 KEYSW, K19 KEYSW, K2 KEYSW, K20 KEYSW, K21 KEYSW, K22 KEYSW, K23 KEYSW, K24 KEYSW, K25 KEYSW, K26 KEYSW, K27 KEYSW, K28 KEYSW, K29 KEYSW, K3 KEYSW, K30 KEYSW, K31 KEYSW, K32 KEYSW, K33 KEYSW, K34 KEYSW, K35 KEYSW, K36 KEYSW, K37 KEYSW, K38 KEYSW, K39 KEYSW, K4 KEYSW, K40 KEYSW, K41 KEYSW, K42 KEYSW, K43 KEYSW, K44 KEYSW, K45 KEYSW, K46 KEYSW, K47 KEYSW, K48 KEYSW, K49 KEYSW, K5 KEYSW, K50 KEYSW, K51 KEYSW, K52 KEYSW, K53 KEYSW, K54 KEYSW, K55 KEYSW, K56 KEYSW, K57 KEYSW, K58 KEYSW, K59 KEYSW, K6 KEYSW, K60 KEYSW, K61 KEYSW, K62 KEYSW, K63 KEYSW, K64 KEYSW, K7 KEYSW, K8 KEYSW, K9 KEYSW, SW0 Reset, U0 ATmega32U2, U1 PRTR5V0U2X, Y0 16MHz

Commit message: fix ISP pins, curved corners, larger component spacing
Parts:
- moved C0 3.37 mm to (181.0, 173.0)
- moved C3 2.38 mm to (154.0, 159.5)
- moved C4 1.59 mm to (157.2, 159.5)
- moved R7 1.59 mm to (78.6, 88.9)
- moved L0 1.59 mm to (98.4, 88.1)
- moved D58 1.02 mm to (246.9, 170.9)
- moved F1 0.79 mm to (100.8, 104.0)
- moved R6 0.79 mm to (81.8, 88.9)
- moved C2 0.79 mm to (164.3, 172.8)
- moved C5 0.79 mm to (160.3, 159.5)
- moved D28 0.76 mm to (127.8, 138.1)
- moved D0 0.76 mm to (113.5, 100.0)
- moved D14 0.76 mm to (123.0, 119.1)
- moved D41 0.76 mm to (137.3, 157.2)
- moved R5 0.73 mm to (177.0, 155.6)
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Connections:
- ISP0 pad 1: COL12 -> COL11
- ISP0 pad 3: COL10 -> COL9
- ISP0 pad 4: COL11 -> COL10
Routing:
- net COL9: track 167.3 -> 182.7 mm, vias 6 -> 8
- net COL12: track 242.5 -> 231.2 mm, vias 8 -> 6
- net GND: track 278.8 -> 289.3 mm
- net Net-(C0-Pad1): track 3.78 -> 7.14 mm
- net COL11: track 219.9 -> 217.8 mm
- net Earth: track 19.8 -> 21.4 mm
- net +5V: track 184.0 -> 185.3 mm
- net D-: track 161.0 -> 159.8 mm
- net COL10: track 200.3 -> 201.3 mm
- net COL14: track 241.1 -> 240.2 mm
- net COL13: track 236.9 -> 236.1 mm
- net VCC: track 33.7 -> 34.5 mm
- net Net-(J0-PadA5): track 12.9 -> 13.6 mm
- net XTAL2: track 11.2 -> 12.0 mm
- net Net-(J0-PadB5): track 20.4 -> 21.2 mm
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Other:
- outline, holes or cut-outs redrawn
- board text added: "exp60 rev 1.1 by Christian Schulze"
- board text removed: "exp60 by Christian Schulze"
